File: jfet-guitar-amp.sch (KiCad schematic (older format))
At the start: 48 parts, among them J1 JST_XH_2, J2 JST_XH_2, J3 JST_XH_3, Q1 J201, Q2 J201, Q3 J201, U1 4580

Commit message: changes to component footprints, new layout WIP
Parts:
- C10: footprint Capacitor_SMD:C_0805_2012Metric -> Capacitor_SMD:CP_Elec_8x6.9; PN (none) -> 124-8280
- C13: renamed from C?; footprint Capacitor_SMD:C_0805_2012Metric -> Capacitor_SMD:CP_Elec_8x6.9; PN (none) -> 124-8280
- J1, J2: footprint Connector_JST:JST_XH_B02B-XH-A_1x02_P2.50mm_Vertical -> Footprints:wire_strainrelief_2
- J3: footprint Connector_JST:JST_XH_B03B-XH-A_1x03_P2.50mm_Vertical -> Footprints:wire_strainrelief_3
- Q1, Q2, Q3: footprint Package_TO_SOT_THT:TO-92 -> Package_TO_SOT_SMD:SOT-23
- gave numbers to parts that had none: 5
Other:
- note added: "MMBF411x?"
Changed lines of the file:
@@
 F 0 "Q1" H 3025 3775 50  0000 L CNN
 F 1 "J201" H 2950 3475 50  0000 L CNN
-F 2 "Package_TO_SOT_THT:TO-92" H 3275 3725 50  0001 C CNN
+F 2 "Package_TO_SOT_SMD:SOT-23" H 3275 3725 50  0001 C CNN
 F 3 "~" H 3075 3625 50  0001 C CNN
 	1    3075 3625
@@
 F 0 "J1" H 1369 3400 50  0000 C CNN
 F 1 "JST_XH_2" H 1369 3491 50  0000 C CNN
-F 2 "Connector_JST:JST_XH_B02B-XH-A_1x02_P2.50mm_Vertical" H 1475 3725 50  0001 C CNN
+F 2 "Footprints:wire_strainrelief_2" H 1475 3725 50  0001 C CNN
 F 3 "~" H 1475 3725 50  0001 C CNN
 	1    1475 3725
@@
 F 0 "Q2" H 3900 3725 50  0000 L CNN
 F 1 "J201" H 3925 3450 50  0000 L CNN
-F 2 "Package_TO_SOT_THT:TO-92" H 4200 3700 50  0001 C CNN
+F 2 "Package_TO_SOT_SMD:SOT-23" H 4200 3700 50  0001 C CNN
 F 3 "~" H 4000 3600 50  0001 C CNN
 	1    4000 3600
@@
 F 0 "Q3" H 5691 3646 50  0000 L CNN
 F 1 "J201" H 5691 3555 50  0000 L CNN
-F 2 "Package_TO_SOT_THT:TO-92" H 5700 3700 50  0001 C CNN
+F 2 "Package_TO_SOT_SMD:SOT-23" H 5700 3700 50  0001 C CNN
 F 3 "~" H 5500 3600 50  0001 C CNN
 	1    5500 3600
@@
 F 0 "J2" H 643 950 50  0000 C CNN
 F 1 "JST_XH_2" H 643 1041 50  0000 C CNN
-F 2 "Connector_JST:JST_XH_B02B-XH-A_1x02_P2.50mm_Vertical" H 750 1275 50  0001 C CNN
+F 2 "Footprints:wire_strainrelief_2" H 750 1275 50  0001 C CNN
 F 3 "~" H 750 1275 50  0001 C CNN
 	1    750  1275
@@
 F 0 "C10" H 3608 1229 50  0000 R CNN
 F 1 "470u" H 3608 1320 50  0000 R CNN
-F 2 "Capacitor_SMD:C_0805_2012Metric" H 3700 1275 50  0001 C CNN
+F 2 "Capacitor_SMD:CP_Elec_8x6.9" H 3700 1275 50  0001 C CNN
 F 3 "~" H 3700 1275 50  0001 C CNN
+F 4 "124-8280" H 3700 1275 50  0001 C CNN "PN"
 	1    3700 1275
 	1    0    0    1
@@
 F 0 "J3" H 8868 2700 50  0000 C CNN
 F 1 "JST_XH_3" H 8868 2791 50  0000 C CNN
-F 2 "Connector_JST:JST_XH_B03B-XH-A_1x03_P2.50mm_Vertical" H 8975 3025 50  0001 C CNN
+F 2 "Footprints:wire_strainrelief_3" H 8975 3025 50  0001 C CNN
 F 3 "~" H 8975 3025 50  0001 C CNN
 	1    8975 3025
@@
 	8300 3025 8775 3025
 $Comp
-L Device:R_Small R?
+L Device:R_Small R14
 U 1 1 5C14A092
 P 8200 2925
-F 0 "R?" V 8275 2925 50  0000 C CNN
+F 0 "R14" V 8275 2925 50  0000 C CNN
 F 1 "120R" V 8350 2925 50  0000 C CNN
 F 2 "Resistor_SMD:R_0805_2012Metric" H 8200 2925 50  0001 C CNN
@@
 $EndComp
 $Comp
-L Device:R_Small R?
+L Device:R_Small R19
 U 1 1 5C14E7AA
 P 8200 3025
-F 0 "R?" V 8275 3025 50  0000 C CNN
+F 0 "R19" V 8275 3025 50  0000 C CNN
 F 1 "120R" V 8350 3025 50  0000 C CNN
 F 2 "Resistor_SMD:R_0805_2012Metric" H 8200 3025 50  0001 C CNN
@@
 	3700 1150 3900 1150
 $Comp
-L Device:C_Small C?
+L Device:C_Small C13
 U 1 1 5C169024
 P 3700 975
-F 0 "C?" H 3608 929 50  0000 R CNN
+F 0 "C13" H 3608 929 50  0000 R CNN
 F 1 "470u" H 3608 1020 50  0000 R CNN
-F 2 "Capacitor_SMD:C_0805_2012Metric" H 3700 975 50  0001 C CNN
+F 2 "Capacitor_SMD:CP_Elec_8x6.9" H 3700 975 50  0001 C CNN
 F 3 "~" H 3700 975 50  0001 C CNN
+F 4 "124-8280" H 3700 975 50  0001 C CNN "PN"
 	1    3700 975
 	1    0    0    1
@@
 	8725 3375 8700 3375
 $Comp
-L Device:C_Small C?
+L Device:C_Small C14
 U 1 1 5C2089A4
 P 5850 4000
-F 0 "C?" H 5800 3925 50  0000 R CNN
+F 0 "C14" H 5800 3925 50  0000 R CNN
 F 1 "10u" H 5800 4075 50  0000 R CNN
 F 2 "Capacitor_SMD:C_0805_2012Metric" H 5850 4000 50  0001 C CNN
@@
 Connection ~ 4300 3375
 $Comp
-L Device:R_Small R?
+L Device:R_Small R11
 U 1 1 5C261ADA
 P 2525 3625
-F 0 "R?" V 2600 3625 50  0000 C CNN
+F 0 "R11" V 2600 3625 50  0000 C CNN
 F 1 "33K" V 2675 3625 50  0000 C CNN
 F 2 "Resistor_SMD:R_0805_2012Metric" H 2525 3625 50  0001 C CNN
@@
 $EndComp
 $Comp
-L Device:C_Small C?
+L Device:C_Small C12
 U 1 1 5C261CF8
 P 2775 3825
-F 0 "C?" H 2700 3850 50  0000 R CNN
+F 0 "C12" H 2700 3850 50  0000 R CNN
 F 1 "220p" H 2725 3950 50  0000 R CNN
 F 2 "Capacitor_SMD:C_0805_2012Metric" H 2775 3825 50  0001 C CNN
@@
 	2775 4150 3175 4150
 Connection ~ 3175 4150
+Text Notes 3025 4450 0    50   ~ 0
+MMBF411x?
 $EndSCHEMATC
