File: _saved_jfet-guitar-amp.sch (KiCad schematic (older format))
At the start: 52 parts, among them J1 Conn_2, J2 Conn_2, J3 Conn_3, Q1 J201, Q2 J201, Q3 J201, U1 4580

Commit message: PCB updated
Parts:
- removed R?: 100K, Resistor_SMD:R_0805_2012Metric, symbol Device:R_Small
- gave numbers to parts that had none: 8
Connections:
- wire segments 168 -> 167
Changed lines of the file:
@@
 MMBF411x?
 $Comp
-L Amplifier_Operational:MCP6001-OT U?
+L Amplifier_Operational:MCP6001-OT U2
 U 1 1 5C198255
 P 5600 1300
-F 0 "U?" H 5700 1450 50  0000 L CNN
+F 0 "U2" H 5700 1450 50  0000 L CNN
 F 1 "TSX9291" H 5625 1100 50  0000 L CNN
 F 2 "Package_TO_SOT_SMD:SOT-23-5" H 5500 1100 50  0001 L CNN
@@
 	5900 1300 5950 1300
 $Comp
-L power:+9V #PWR?
+L power:+9V #PWR0104
 U 1 1 5C1B726E
 P 5500 700
-F 0 "#PWR?" H 5500 550 50  0001 C CNN
+F 0 "#PWR0104" H 5500 550 50  0001 C CNN
 F 1 "+9V" H 5515 873 50  0000 C CNN
 F 2 "" H 5500 700 50  0001 C CNN
@@
 $EndComp
 $Comp
-L power:GND #PWR?
+L power:GND #PWR0105
 U 1 1 5C1B72D5
 P 5500 1750
-F 0 "#PWR?" H 5500 1500 50  0001 C CNN
+F 0 "#PWR0105" H 5500 1500 50  0001 C CNN
 F 1 "GND" H 5505 1577 50  0000 C CNN
 F 2 "" H 5500 1750 50  0001 C CNN
@@
 	5500 700  5500 725
 $Comp
-L Device:C_Small C?
+L Device:C_Small C10
 U 1 1 5C1C5ED8
 P 5575 850
-F 0 "C?" H 5483 804 50  0000 R CNN
+F 0 "C10" H 5483 804 50  0000 R CNN
 F 1 "100n" H 5483 895 50  0000 R CNN
 F 2 "Capacitor_SMD:C_0805_2012Metric" H 5575 850 50  0001 C CNN
@@
 	5500 725  5500 1000
 $Comp
-L power:GND #PWR?
+L power:GND #PWR0106
 U 1 1 5C1CF888
 P 5575 975
-F 0 "#PWR?" H 5575 725 50  0001 C CNN
+F 0 "#PWR0106" H 5575 725 50  0001 C CNN
 F 1 "GND" H 5700 900 50  0000 C CNN
 F 2 "" H 5575 975 50  0001 C CNN
@@
 	5575 975  5575 950
 $Comp
-L Device:R_Small R?
+L Device:R_Small R1
 U 1 1 5C1D4DE0
 P 4975 950
-F 0 "R?" H 4917 904 50  0000 R CNN
+F 0 "R1" H 4917 904 50  0000 R CNN
 F 1 "100K" H 4917 995 50  0000 R CNN
 F 2 "Resistor_SMD:R_0805_2012Metric" H 4975 950 50  0001 C CNN
@@
 $EndComp
 $Comp
-L Device:R_Small R?
+L Device:R_Small R2
 U 1 1 5C1D50BA
 P 4975 1500
-F 0 "R?" H 4917 1454 50  0000 R CNN
+F 0 "R2" H 4917 1454 50  0000 R CNN
 F 1 "100K" H 4917 1545 50  0000 R CNN
 F 2 "Resistor_SMD:R_0805_2012Metric" H 4975 1500 50  0001 C CNN
@@
 Wire Wire Line
 	4975 1050 4975 1200
-$Comp
-L Device:R_Small R?
-U 1 1 5C2022EA
-P 5150 1200
-F 0 "R?" V 5075 1275 50  0000 R CNN
-F 1 "100K" V 5000 1275 50  0000 R CNN
-F 2 "Resistor_SMD:R_0805_2012Metric" H 5150 1200 50  0001 C CNN
-F 3 "~" H 5150 1200 50  0001 C CNN
-	1    5150 1200
-	0    -1   1    0
-$EndComp
-Wire Wire Line
-	5050 1200 4975 1200
 Connection ~ 4975 1200
 Wire Wire Line
 	4975 1200 4975 1400
-Wire Wire Line
-	5250 1200 5300 1200
-$Comp
-L Device:R_Small R?
+$Comp
+L Device:R_Small R21
 U 1 1 5C21C398
 P 7250 950
-F 0 "R?" H 7192 904 50  0000 R CNN
+F 0 "R21" H 7192 904 50  0000 R CNN
 F 1 "4K7" H 7192 995 50  0000 R CNN
 F 2 "Resistor_SMD:R_0805_2012Metric" H 7250 950 50  0001 C CNN
@@
 $EndComp
 $Comp
-L Device:R_Small R?
+L Device:R_Small R22
 U 1 1 5C21C462
 P 7250 1250
-F 0 "R?" H 7192 1204 50  0000 R CNN
+F 0 "R22" H 7192 1204 50  0000 R CNN
 F 1 "4K7" H 7192 1295 50  0000 R CNN
 F 2 "Resistor_SMD:R_0805_2012Metric" H 7250 1250 50  0001 C CNN
@@
 $EndComp
 $Comp
-L Device:C_Small C?
+L Device:C_Small C11
 U 1 1 5C21C79A
 P 7625 950
-F 0 "C?" H 7533 904 50  0000 R CNN
+F 0 "C11" H 7533 904 50  0000 R CNN
 F 1 "470u" H 7533 995 50  0000 R CNN
 F 2 "Capacitor_SMD:C_Elec_8x6.2" H 7625 950 50  0001 C CNN
@@
 $EndComp
 $Comp
-L Device:C_Small C?
+L Device:C_Small C13
 U 1 1 5C21C8DD
 P 7625 1250
-F 0 "C?" H 7533 1204 50  0000 R CNN
+F 0 "C13" H 7533 1204 50  0000 R CNN
 F 1 "470u" H 7533 1295 50  0000 R CNN
 F 2 "Capacitor_SMD:C_Elec_8x6.2" H 7625 1250 50  0001 C CNN
@@
 	7250 1100 7250 1150
 $Comp
-L power:+9V #PWR?
+L power:+9V #PWR0107
 U 1 1 5C243C02
 P 7250 725
-F 0 "#PWR?" H 7250 575 50  0001 C CNN
+F 0 "#PWR0107" H 7250 575 50  0001 C CNN
 F 1 "+9V" H 7265 898 50  0000 C CNN
 F 2 "" H 7250 725 50  0001 C CNN
@@
 Connection ~ 7250 775
 $Comp
-L power:GND #PWR?
+L power:GND #PWR0108
 U 1 1 5C24AA1F
 P 7250 1450
-F 0 "#PWR?" H 7250 1200 50  0001 C CNN
+F 0 "#PWR0108" H 7250 1200 50  0001 C CNN
 F 1 "GND" H 7255 1277 50  0000 C CNN
 F 2 "" H 7250 1450 50  0001 C CNN
@@
 Text Notes 5700 1750 0    50   ~ 0
 Choice of either op amp or resistor virtual ground
+Wire Wire Line
+	4975 1200 5300 1200
 $EndSCHEMATC
